File: radio.sch (KiCad schematic (older format))
At the start: 85 parts, among them P1 CONN_01X02, P2 CONN_01X02, P3 CONN_01X02, P4 CONN_01X10, P5 CONN_01X02, P6 CONN_01X02, P8 CONN_01X02, U1 MAX2870, U2 ADL5380, U3 ADL5375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

Commit message: Values set up correctly
Parts:
- C31, C32, C36: value C -> 1u
- C34: value C -> 840p
- C35, C38: value C -> 0.1u
- C37: value C -> 12n
- R12: value R -> 240
- R7: value R -> 5.1k
Changed lines of the file:
@@
 LIBS:elepaja
 LIBS:sma_edge
-LIBS:radio-cache
 EELAYER 25 0
 EELAYER END
@@
 P 2350 2400
 F 0 "C31" H 2375 2500 50  0000 L CNN
-F 1 "C" H 2375 2300 50  0000 L CNN
+F 1 "1u" H 2375 2300 50  0000 L CNN
 F 2 "Capacitors_SMD:C_0805" H 2388 2250 50  0001 C CNN
 F 3 "" H 2350 2400 50  0000 C CNN
@@
 P 2650 2400
 F 0 "C32" H 2675 2500 50  0000 L CNN
-F 1 "C" H 2675 2300 50  0000 L CNN
+F 1 "1u" H 2675 2300 50  0000 L CNN
 F 2 "Capacitors_SMD:C_0805" H 2688 2250 50  0001 C CNN
 F 3 "" H 2650 2400 50  0000 C CNN
@@
 P 3100 2400
 F 0 "C34" H 3125 2500 50  0000 L CNN
-F 1 "C" H 3125 2300 50  0000 L CNN
+F 1 "840p" H 3125 2300 50  0000 L CNN
 F 2 "Capacitors_SMD:C_0805" H 3138 2250 50  0001 C CNN
 F 3 "" H 3100 2400 50  0000 C CNN
@@
 P 3400 2400
 F 0 "C36" H 3425 2500 50  0000 L CNN
-F 1 "C" H 3425 2300 50  0000 L CNN
+F 1 "1u" H 3425 2300 50  0000 L CNN
 F 2 "Capacitors_SMD:C_0805" H 3438 2250 50  0001 C CNN
 F 3 "" H 3400 2400 50  0000 C CNN
@@
 P 2900 2400
 F 0 "R7" V 2980 2400 50  0000 C CNN
-F 1 "R" V 2900 2400 50  0000 C CNN
+F 1 "5.1k" V 2900 2400 50  0000 C CNN
 F 2 "Resistors_SMD:R_0805" V 2830 2400 50  0001 C CNN
 F 3 "" H 2900 2400 50  0000 C CNN
@@
 P 3400 2050
 F 0 "R12" V 3480 2050 50  0000 C CNN
-F 1 "R" V 3400 2050 50  0000 C CNN
+F 1 "240" V 3400 2050 50  0000 C CNN
 F 2 "Resistors_SMD:R_0805" V 3330 2050 50  0001 C CNN
 F 3 "" H 3400 2050 50  0000 C CNN
@@
 P 3250 5100
 F 0 "C35" H 3275 5200 50  0000 L CNN
-F 1 "C" H 3275 5000 50  0000 L CNN
+F 1 "0.1u" H 3275 5000 50  0000 L CNN
 F 2 "Capacitors_SMD:C_0805" H 3288 4950 50  0001 C CNN
 F 3 "" H 3250 5100 50  0000 C CNN
@@
 P 3450 5200
 F 0 "C37" H 3475 5300 50  0000 L CNN
-F 1 "C" H 3475 5100 50  0000 L CNN
+F 1 "12n" H 3475 5100 50  0000 L CNN
 F 2 "Capacitors_SMD:C_0805" H 3488 5050 50  0001 C CNN
 F 3 "" H 3450 5200 50  0000 C CNN
@@
 P 3700 4950
 F 0 "C38" H 3725 5050 50  0000 L CNN
-F 1 "C" H 3725 4850 50  0000 L CNN
+F 1 "0.1u" H 3725 4850 50  0000 L CNN
 F 2 "Capacitors_SMD:C_0805" H 3738 4800 50  0001 C CNN
 F 3 "" H 3700 4950 50  0000 C CNN
