File: radio.kicad_pcb (KiCad board)
At the start: 2 copper layers, 50.8 x 50.8 mm, 85 parts, among them P1 CONN_01X02, P2 CONN_01X02, P3 CONN_01X02, P4 CONN_01X10, P5 CONN_01X02, P6 CONN_01X02, P8 CONN_01X02, U1 MAX2870, U2 ADL5380, U3 ADL5375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

Commit message: Values set up correctly
Routing:
- net Net-(C25-Pad1): track 19.7 -> 5.50 mm, vias 2 -> 0
- net /VCC_PLL: track 36.9 -> 47.6 mm
- net GND: track 80.6 -> 87.1 mm

Commit message: Adjusted routes
Parts:
- removed W1, W2, W3, W4: TEST_1P, Mounting_Holes:MountingHole_2.2mm_M2
- moved C35 1.71 mm to (163.2, 107.0)
- moved C37 1.56 mm to (164.8, 107.0)
- moved C38 1.41 mm to (166.2, 107.0)
Routing:
- net GND: track 87.1 -> 90.7 mm
- net Net-(C26-Pad1): track 6.95 -> 4.66 mm
- net /MOD_N: track 18.2 -> 16.1 mm
- net Net-(C35-Pad2): track 1.68 -> 3.42 mm
- net /MOD_I_N: track 16.3 -> 18.0 mm
- net Net-(C35-Pad1): track 29.7 -> 31.3 mm
- net /MOD_I_P: track 15.6 -> 17.2 mm
- net /MOD_Q_N: track 16.3 -> 17.6 mm
- net /MOD_Q_P: track 15.6 -> 16.8 mm
- net Net-(C26-Pad2): track 2.99 -> 3.53 mm
Other:
- net class Default: clearance 0.15 -> 0.08; trace_width 0.25 -> 0.4
- rule trace_clearance: 0.15 -> 0.08
